File: el-driver.sch (KiCad schematic (older format))
At the start: 37 parts, among them J1 Conn_01x03, J2 Conn_01x02, Q1 SI3493DDV-T1-GE3, Q2 BSS138, Q3 BSS214NW, Q4 BSS214NW, T1 42XL003-RC, U1 NE555D

Commit message: Version 2.0.0
Signed-off-by: Aaron Williams <aaron.w2@gmail.com>
Parts:
- removed C11: 10uF, Capacitor_SMD:C_0603_1608Metric, symbol Device:C
- removed C12: 1uF, Capacitor_SMD:C_0603_1608Metric, symbol Device:C
- removed C6: 4.7nF, Capacitor_SMD:C_0603_1608Metric, symbol Device:C
- removed C7, C8: 1nF, Capacitor_SMD:C_0603_1608Metric, symbol Device:C
- removed D2: SS24FL, Diode_SMD:D_SOD-123, symbol Aaron:SS24FL
- removed Q1: SI3493DDV-T1-GE3, Package_TO_SOT_SMD:SOT-23-6, symbol Aaron:SI3493DDV-T1-GE3
- removed Q2: BSS138, Package_TO_SOT_SMD:SOT-23, symbol Transistor_FET:BSS138
- removed Q4: BSS214NW, Package_TO_SOT_SMD:SOT-323_SC-70, symbol Transistor_FET:BSS214NW
- removed R1, R2, R5: 100k, Resistor_SMD:R_0603_1608Metric, symbol Device:R
- removed R4: 39.2, Resistor_SMD:R_0603_1608Metric, symbol Device:R
- removed T1: 42XL003-RC, Aaron:Transformer_42XL_EI-14, symbol Device:Transformer_SP_1S
- added TR1: Transformer-EI14, Aaron:Transformer_42XL_EI-14, symbol Aaron:Transformer-EI14
- renumbered C9 to C6, C10 to C7, D3 to D2, J2 to J1, J1 to J2, Q3 to Q1, R8 to R1, R3 to R2, R6 to R3, R7 to R4
Connections:
- net +5V: now also C1.1, C2.1, D2.2 (A), U1.8 (VCC), TR1.3
- net EN: now also U1.4 (R)
- net GND: no longer R1.2
- net at D1.2 (A), Q1.3 (D), R2.1: now also R1.2, TR1.1
- net at J1.2 (Pin_2): now also TR1.6
- net at J1.1 (Pin_1): now also TR1.4
- removed net 5V_SW: C1.1, C2.1, D2.2 (A), U1.4 (R), U1.8 (VCC)
- no-connect marks 0 -> 2
Other:
- moved on the sheet: C3, C4, C5, D1, D2, J1, J2, R1, R2
